Commit message: 1217暂存

File: test_ctrl_ros2/models/test2/mini_model.urdf (robot description, URDF)
Before this commit: robot test2, 4 links, 4 joints
Joints:
- joint force1: limit (none) -> lower=-3.14159 upper=3.14159 effort=10.0 velocity=10.0
- joint no_force1: limit (none) -> lower=-3.14159 upper=3.14159 effort=10.0 velocity=10.0
- joint no_force2: limit (none) -> lower=-3.14159 upper=3.14159 effort=10.0 velocity=10.0
- joint no_force3: limit (none) -> lower=-3.14159 upper=3.14159 effort=10.0 velocity=10.0

Commit message: 251220-四连杆控制demo基本完成

File: test_ctrl_ros2/models/test2/mini_model.urdf (robot description, URDF)
Before this commit: robot test2, 4 links, 4 joints
Links:
- added link link_dummy
Joints:
- joint no_force3: child base_link -> link_dummy

Commit message: 251221-Demo微调

File: test_ctrl_ros2/models/test2/mini_model.urdf (robot description, URDF)
Before this commit: robot test2, 5 links, 4 joints
Joints:
- joint force1: origin (none) -> xyz=0 0 0 rpy=0 0 0
- joint no_force1: origin (none) -> xyz=0.01109 0.038432 0 rpy=0 0 0
- joint no_force2: origin (none) -> xyz=0.071655 0.035574 0 rpy=0 0 0
- joint no_force3: origin (none) -> xyz=0.067254 -0.074006 0 rpy=0 0 0
