Commit message: 260104-初步解决模型坍塌问题，修改好SDF文件并联机构

File: pipe_robot_ros2/models/pipe_robot/pipe_robot.urdf (robot description, URDF)
Before this commit: robot pipe_robot, 53 links, 52 joints
Links:
- added link world
Joints:
- added joint fixed: type fixed, parent world, child BM_01_link
- joint joint_04_10_RN: origin xyz=0.0002000000000002 0.138 0.0455144934992005 rpy=3.14159265358979 -1.5707963267949 0 -> xyz=0.0002000000000002 0.138 0.0455144934992005 rpy=0 -1.5707963267949 0
- joint joint_04_11_RN: origin xyz=-0.000199999999999756 -0.138 0.0455144934992005 rpy=3.14159265358979 -1.5707963267949 0 -> xyz=-0.000199999999999756 -0.138 0.0455144934992005 rpy=0 -1.5707963267949 0
- joint joint_07_08_RF: origin xyz=0 0 0.019 rpy=3.14159265358979 -1.5707963267949 0 -> xyz=0 0 0.019 rpy=3.14159265358979 1.5707963267949 0
- joint joint_24_25_FN: origin xyz=-0.0128898186140129 0.11 -0.07 rpy=1.5707963267949 1.5707963267949 0 -> xyz=-0.0128898186140129 0.11 -0.07 rpy=1.5707963267949 1.5707963267949 3.141592654
- joint joint_24_30_RF: origin xyz=0.084 0.062 -0.07 rpy=3.1416 -1.5708 0 -> xyz=0.084 0.062 -0.07 rpy=0 -1.5708 0
- joint joint_27_32_RN: origin xyz=0.0001999999999997 0.138 0.0455144934992005 rpy=0 -1.5707963267949 0 -> xyz=0.0001999999999997 0.138 0.0455144934992005 rpy=3.14159265358979 -1.5707963267949 0
- joint joint_30_31_RF: origin xyz=0 0 0.019 rpy=3.1416 -1.5708 0 -> xyz=0 0 0.019 rpy=0 1.5708 3.141592654
