Commit message: 260113-修改了原始URDF模型镜像问题，并调整了轮轴正方向

File: URDF/pipe_robot/urdf/pipe_robot.urdf (robot description, URDF)
Before this commit: robot pipe_robot, 53 links, 52 joints
Joints:
- joint joint_01_04_LF: axis 0 0 -1 -> 0 0 1; limit lower=0 upper=0 effort=0 velocity=0 -> lower=-0.0385 upper=0.015 effort=0 velocity=0
- joint joint_01_07_RF: axis 0 0 -1 -> 0 0 1
- joint joint_01_09_RF: axis 0 0 -1 -> 0 0 1; limit (none) -> lower=-0.488692 upper=1.047197533 effort=600 velocity=0.5; type continuous -> revolute
- joint joint_04_10_RN: origin xyz=0.0002000000000002 0.138 0.0455144934992005 rpy=3.14159265358979 -1.5707963267949 0 -> xyz=0.0002000000000002 0.138 0.0455144934992005 rpy=0 -1.5707963267949 0
- joint joint_04_11_RN: origin xyz=-0.000199999999999756 -0.138 0.0455144934992005 rpy=3.14159265358979 -1.5707963267949 0 -> xyz=-0.000199999999999756 -0.138 0.0455144934992005 rpy=0.0 -1.5707963267949 0
- joint joint_05_14_RF: limit (none) -> lower=-0.488692 upper=1.274090 effort=600 velocity=0.8; type continuous -> revolute
- joint joint_06_15_RF: limit (none) -> lower=-0.488692 upper=1.274090 effort=600 velocity=0.8; type continuous -> revolute
- joint joint_07_08_RF: origin xyz=0 0 0.019 rpy=3.14159265358979 -1.5707963267949 0 -> xyz=0 0 0.019 rpy=3.14159265358979 1.5707963267949 0
- joint joint_09_24_RF: limit (none) -> lower=-0.488692 upper=1.047197533 effort=600 velocity=0.5; type continuous -> revolute
- joint joint_10_12_LF: axis 0 0 -1 -> 0 0 1; limit lower=0 upper=0 effort=0 velocity=0 -> lower=-0.011 upper=0 effort=360 velocity=0.06
- joint joint_11_13_LF: axis 0 0 -1 -> 0 0 1; limit lower=0 upper=0 effort=0 velocity=0 -> lower=-0.011 upper=0 effort=360 velocity=0.06
- joint joint_16_20_RF: axis 0 0 -1 -> 0 0 1
- joint joint_17_21_RF: axis 0 0 -1 -> 0 0 1
- joint joint_21_23_RF: axis 0 0 -1 -> 0 0 1
- joint joint_24_27_LF: axis 0 0 -1 -> 0 0 1; limit lower=0 upper=0 effort=0 velocity=0 -> lower=-0.0385 upper=0.015 effort=3000 velocity=0.05
- joint joint_24_30_RF: origin xyz=0.084 0.062 -0.07 rpy=3.1416 -1.5708 0 -> xyz=0.084 0.062 -0.07 rpy=3.1416 -1.5708 3.14159
- joint joint_27_32_RN: origin xyz=0.0001999999999997 0.138 0.0455144934992005 rpy=0 -1.5707963267949 0 -> xyz=0.0001999999999997 0.138 0.0455144934992005 rpy=3.14159 -1.5707963267949 0
- joint joint_28_36_RF: limit (none) -> lower=-0.488692 upper=1.274090 effort=600 velocity=0.8; type continuous -> revolute
- joint joint_29_37_RF: limit (none) -> lower=-0.488692 upper=1.274090 effort=600 velocity=0.8; type continuous -> revolute
- joint joint_30_31_RF: axis 0 0 -1 -> 0 0 1; origin xyz=0 0 0.019 rpy=3.1416 -1.5708 0 -> xyz=0 0 0.019 rpy=3.1416 1.5708 0
- joint joint_32_34_LF: axis 0 0 -1 -> 0 0 1; limit lower=0 upper=0 effort=0 velocity=0 -> lower=-0.011 upper=0 effort=360 velocity=0.06
- joint joint_33_35_LF: axis 0 0 -1 -> 0 0 1; limit lower=0 upper=0 effort=0 velocity=0 -> lower=-0.011 upper=0 effort=360 velocity=0.06
- joint joint_38_42_RF: axis 0 0 -1 -> 0 0 1
- joint joint_39_43_RF: axis 0 0 -1 -> 0 0 1
- joint joint_42_44_RF: axis 0 0 -1 -> 0 0 1
